File: Hardware/KiCad_ArduinoUnoR3ProtoShield/KiCad_ArduinoUnoR3ProtoShield.kicad_pcb (KiCad board)
At the start: 2 copper layers, 68.6 x 53.3 mm, 8 parts, among them P1 Power, P2 Analog, P3 Digital, P4 Digital, P5 CONN_01X01, P6 CONN_01X01, P7 CONN_01X01, P8 CONN_01X01

Commit message: added all parts
Parts:
- added Piezzo: PIEZO-MCKPI-G1410, myKiCadLib:PIEZO-MCKPI-G1410, F.Cu at (144.0, 101.0)
- added R4,7k: R_Axial_DIN0207_L6.3mm_D2.5mm_P15.24mm_Horizontal, Resistor_THT:R_Axial_DIN0207_L6.3mm_D2.5mm_P15.24mm_Horizontal, F.Cu at (131.3, 106.0)
- added Stereo Buchse 3,5mm: EAR, myKiCadLib:Tayda_3.5mm_stereo_TRS_jack_A-853, F.Cu at (116.1, 118.7)
- added TR433MHz: RF_Transmitter_433_MHz, myKiCadLib:RF_Transmitter_433_MHz, F.Cu at (159.3, 101.0)
Connections:
- net /10(**/SS) renamed /10(**/SS)
- net /11(**/MOSI) renamed /11(**/MOSI)
- P1 pad 1: Net-(P1-Pad1) -> unconnected-(P1-Pad1)
- P5 pad 1: Net-(P5-Pad1) -> unconnected-(P5-Pad1)
- P6 pad 1: Net-(P6-Pad1) -> unconnected-(P6-Pad1)
- P7 pad 1: Net-(P7-Pad1) -> unconnected-(P7-Pad1)
- P8 pad 1: Net-(P8-Pad1) -> unconnected-(P8-Pad1)
